Commit message: added aruco code but not working

File: urdf/ur5.urdf (robot description, URDF)
Before this commit: robot ur5_robot, 12 links, 11 joints
Links:
- added link box_link, mass 0.1; collision box size=1 1 0.001; visual box size=1 1 0.001
- added link camera_link, mass 1e-5; collision box size=0.05 0.05 0.05; visual box size=0.05 0.05 0.05
Joints:
- added joint box_link_joint: type fixed, parent base_link, child box_link, origin xyz=0 0 -0.1 rpy=0 0 0
- added joint camera_joint: type fixed, parent tool0, child camera_link, origin xyz=0 0 0 rpy=0 -1.57 0, axis 0 1 0

Commit message: adding gazebo joint control drivers and also correct some bugs for motion planning

File: urdf/ur5.urdf (robot description, URDF)
Before this commit: robot ur5_robot, 14 links, 13 joints
Links:
- link box_link: geometry visual box size=1 1 0.001
Joints:
- joint base_link_world: origin xyz=0 0 1 rpy=0 0 0 -> xyz=0 0 0 rpy=0 0 0

Commit message: still need to modify about quaternion

File: urdf/ur5.urdf (robot description, URDF)
Before this commit: robot ur5_robot, 14 links, 13 joints
Links:
- link box_link: geometry collision box size=1 1 0.0001; visual box size=1 1 0.0001
Joints:
- joint base_link_world: origin xyz=0 0 0 rpy=0 0 0 -> xyz=0 0 0.2 rpy=0 0 0

Commit message: right pose wrong orientation

File: urdf/ur5.urdf (robot description, URDF)
Before this commit: robot ur5_robot, 14 links, 13 joints
Links:
- removed link box_link
Joints:
- removed joint box_link_joint

Commit message: get data

File: urdf/ur5.urdf (robot description, URDF)
Before this commit: robot ur5_robot, 13 links, 12 joints
Links:
- added link box_link, mass 0.1; collision box size=1 1 0.0001; visual box size=1 1 0.0001
Joints:
- added joint box_link_joint: type fixed, parent base_link, child box_link, origin xyz=0 0 -0.1 rpy=0 0 0
